Commit message: assemble scans progress
the scans are being assembled and published into the base_link frame but they just need to be offset by the final arm pose

File: abb_irb1600_6_145_support/urdf/irb1600_6_145_macro.xacro (robot description, xacro)
@@ -139,5 +139,5 @@
     <child link="${prefix}link_3"/>
     <axis xyz="0 1 0"/>
-    <limit lower="-4.1015" upper="0.9599" effort="0" velocity="2.9670"/>
+    <limit lower="-0.349" upper="0.9599" effort="0" velocity="2.9670"/>
   </joint>
   <joint name="${prefix}joint_4" type="revolute">

Commit message: test

File: abb_irb1600_6_145_support/urdf/irb1600_6_145_macro.xacro (robot description, xacro)
@@ -139,5 +139,5 @@
     <child link="${prefix}link_3"/>
     <axis xyz="0 1 0"/>
-    <limit lower="-4.1015" upper="0.9599" effort="0" velocity="2.9670"/>
+    <limit lower="-0.349" upper="0.9599" effort="0" velocity="2.9670"/>
   </joint>
   <joint name="${prefix}joint_4" type="revolute">
@@ -160,5 +160,5 @@
     <child link="${prefix}link_6"/>
     <axis xyz="1 0 0"/>
-    <limit lower="-6.9813" upper="6.9813" effort="0" velocity="7.854"/>
+    <limit lower="-3.14159" upper="3.14159" effort="0" velocity="7.854"/>
   </joint>
   <!-- end of joint list -->
